Commit message: chore(alohamini): refresh generated kinematics assets

File: src/lerobot/robots/alohamini/assets/alohamini2pro/alohamini2pro_kinematic.urdf (robot description, URDF)
Before this commit: robot alohamini2pro_kinematic, 31 links, 30 joints
Joints:
- joint left_elbow_flex: limit lower=-0.0703594430376 upper=3.22002934698 effort=2.3 velocity=4 -> lower=-0.0703594430376 upper=3.22002934698 effort=2.21 velocity=2.48
- joint left_shoulder_lift: limit lower=-3.29519440558 upper=0.160864309523 effort=2.3 velocity=4 -> lower=-3.29519440558 upper=0.160864309523 effort=2.21 velocity=2.48
- joint right_elbow_flex: limit lower=-0.0703594430376 upper=3.22002934698 effort=2.3 velocity=4 -> lower=-0.0703594430376 upper=3.22002934698 effort=2.21 velocity=2.48
- joint right_shoulder_lift: limit lower=-3.29519440558 upper=0.160864309523 effort=2.3 velocity=4 -> lower=-3.29519440558 upper=0.160864309523 effort=2.21 velocity=2.48
- joint vertical_move: limit lower=-0.3 upper=0.3 effort=77 velocity=0.08 -> lower=-0.3 upper=0.3 effort=74.2 velocity=0.05

File: src/lerobot/robots/alohamini/assets/alohamini2pro/alohamini2pro_left_kinematic.urdf (robot description, URDF)
Before this commit: robot alohamini2pro_left_kinematic, 10 links, 9 joints
Joints:
- joint left_elbow_flex: limit lower=-0.0703594430376 upper=3.22002934698 effort=2.3 velocity=4 -> lower=-0.0703594430376 upper=3.22002934698 effort=2.21 velocity=2.48
- joint left_shoulder_lift: limit lower=-3.29519440558 upper=0.160864309523 effort=2.3 velocity=4 -> lower=-3.29519440558 upper=0.160864309523 effort=2.21 velocity=2.48

File: src/lerobot/robots/alohamini/assets/alohamini2pro/alohamini2pro_right_kinematic.urdf (robot description, URDF)
Before this commit: robot alohamini2pro_right_kinematic, 10 links, 9 joints
Joints:
- joint right_elbow_flex: limit lower=-0.0703594430376 upper=3.22002934698 effort=2.3 velocity=4 -> lower=-0.0703594430376 upper=3.22002934698 effort=2.21 velocity=2.48
- joint right_shoulder_lift: limit lower=-3.29519440558 upper=0.160864309523 effort=2.3 velocity=4 -> lower=-3.29519440558 upper=0.160864309523 effort=2.21 velocity=2.48

Commit message: feat(alohamini): add MoveIt and guarded ROS 2 control

File: src/lerobot/robots/alohamini/assets/alohamini2pro/alohamini2pro_kinematic.urdf (robot description, URDF)
Before this commit: robot alohamini2pro_kinematic, 31 links, 30 joints
Joints:
- joint left_shoulder_pan: limit lower=-2.23961195031 upper=2.13376727595 effort=1.57 velocity=4.2 -> lower=-2.13376727595 upper=2.23961195031 effort=1.57 velocity=4.2
- joint right_shoulder_pan: limit lower=-2.23961195031 upper=2.13376727595 effort=1.57 velocity=4.2 -> lower=-2.13376727595 upper=2.23961195031 effort=1.57 velocity=4.2

File: src/lerobot/robots/alohamini/assets/alohamini2pro/alohamini2pro_left_kinematic.urdf (robot description, URDF)
Before this commit: robot alohamini2pro_left_kinematic, 10 links, 9 joints
Joints:
- joint left_shoulder_pan: limit lower=-2.23961195031 upper=2.13376727595 effort=1.57 velocity=4.2 -> lower=-2.13376727595 upper=2.23961195031 effort=1.57 velocity=4.2

File: src/lerobot/robots/alohamini/assets/alohamini2pro/alohamini2pro_right_kinematic.urdf (robot description, URDF)
Before this commit: robot alohamini2pro_right_kinematic, 10 links, 9 joints
Joints:
- joint right_shoulder_pan: limit lower=-2.23961195031 upper=2.13376727595 effort=1.57 velocity=4.2 -> lower=-2.13376727595 upper=2.23961195031 effort=1.57 velocity=4.2
